File: flash_sar_adc/flash_sar_adc/flash_sar_adc.kicad_pcb (KiCad board)
At the start: 2 copper layers, 40 x 75 mm, 70 parts, among them J1 Conn_02x06_Matched, J2 Conn_02x06_Matched, U1 LM339DR, U10 RH-5000, U2 LM339DR, U3 OPA843xDBV, U4 SPX3819M5-L-3-0, U5 HL-BNC-KHDA, U6 RH-5000, U7 HL-BNC-KHDA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

Commit message: fixed power supply errors
Parts:
- removed C1: 10nF, PCM_JLCPCB:C_0402
- removed C5: 1uF, PCM_JLCPCB:C_0402
- removed C9: 100nF, PCM_JLCPCB:C_0402
- removed R34: 1kΩ, PCM_JLCPCB:R_0402
- removed U4: SPX3819M5-L-3-0, Package_TO_SOT_SMD:SOT-23-5
- U1, U2: value LM339DR -> LM339LVDR
Connections:
- C10 pad 1: +5V -> +3V3
- C2 pad 1: +5V -> +3V3
- C3 pad 1: +5V -> +3V3
- J1 pad 12: +5V -> +3V3
- J1 pad 6: +5V -> +3V3
- J2 pad 12: +5V -> +3V3
- J2 pad 6: +5V -> +3V3
- U1 pad 3: +5V -> +3V3
- U2 pad 3: +5V -> +3V3
- U3 pad 5: +5V -> +3V3
Routing:
- net +5V: track 93.4 -> 0.00 mm
- net +3V3: track 29.5 -> 119.5 mm
- net GND: track 13.4 -> 10.0 mm, vias 16 -> 11
- net Net-(U4-BP): track 1.81 -> 0.00 mm
Other:
- board text added: "3V3 3V3"
- board text removed: "+5V +5V"

Commit message: added version number
Other:
- board text added: "V1.0"
Changed lines of the file:
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@@
+		)
+	)
+	(gr_text "V1.0"
+		(at 30.675 62.3 90)
+		(layer "F.SilkS")
+		(effects
+			(font
+				(size 1 1)
+				(thickness 0.15)
+			)
+			(justify bottom)
 		)
 	)

Commit message: fixed a few more silkscreen errors
Parts:
- U3: value OPA843xDBV -> COS8051SOT
- moved G*** 0.20 mm to (57.4, 60.4)
